File: Color-Experimentation.sch (EAGLE design)
At the start: 24 parts, among them J1 10118193-0001LF, U2 ATTINY85-20MUR

Commit message: Use LBR, cleanup, export Bill of Materials
Parts:
- BLUE, GREEN, MIXED, RED: value WS2812_5050 -> WS2812; device SparkFun-LED:WS2812_5050 -> Color-Experimentation:WS2812_5050
- BLUE_POT, GREEN_POT, RED_POT: value PTA2043-2015DPB103 -> 10k; device BoardLE+:PTA2043-2015DPB103 -> Color-Experimentation:PTA2043-2015DPB103
- C1, C3, C4, C5, C6: device BoardLE+:CAP_0.1UF_25V_X7R-0603 -> Color-Experimentation:CAP_0.1UF_25V_X7R-0603
- C2: device BoardLE+:CAP_22UF_16V_X5R-0603 -> Color-Experimentation:CAP_22UF_16V_X5R-0603
- GND, MISO, MOSI, RST, SCK, VCC: device DoggBone_RC5:TEST-POINT40MIL -> Color-Experimentation:TEST-POINT40MIL
- J1: device BoardLE+:10118193-0001LF -> Color-Experimentation:10118193-0001LF
- J2: device BoardLE+:CONN_02 -> Color-Experimentation:CONN_02
- JP1, JP2: device DoggBone_RC5:JUMPER-SMT_2_NO_SILK -> Color-Experimentation:JUMPER-SMT_2_NO_SILK
- U2: device DoggBone_RC5:ATTINY85-20MUR -> Color-Experimentation:ATTINY85-20MUR
Changed lines of the file:
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@@
 </attributes>
 <variantdefs>
+<variantdef name="DEFAULT"/>
 </variantdefs>
 <classes>
@@
 </classes>
 <parts>
-<part name="U2" library="DoggBone_RC5" library_urn="urn:adsk.eagle:library:25643843" deviceset="ATTINY85-20MUR" device="" package3d_urn="urn:adsk.eagle:package:30179417/2"/>
-<part name="GND14" library="BoardLE+" library_urn="urn:adsk.eagle:library:23298109" deviceset="GND" device=""/>
-<part name="SUPPLY1" library="DoggBone_RC5" library_urn="urn:adsk.eagle:library:25643843" deviceset="V_USB" device=""/>
-<part name="SCK" library="DoggBone_RC5" library_urn="urn:adsk.eagle:library:25643843" deviceset="TEST-POINT" device="40MIL" package3d_urn="urn:adsk.eagle:package:25643991/1"/>
-<part name="MOSI" library="DoggBone_RC5" library_urn="urn:adsk.eagle:library:25643843" deviceset="TEST-POINT" device="40MIL" package3d_urn="urn:adsk.eagle:package:25643991/1"/>
-<part name="MISO" library="DoggBone_RC5" library_urn="urn:adsk.eagle:library:25643843" deviceset="TEST-POINT" device="40MIL" package3d_urn="urn:adsk.eagle:package:25643991/1"/>
-<part name="RST" library="DoggBone_RC5" library_urn="urn:adsk.eagle:library:25643843" deviceset="TEST-POINT" device="40MIL" package3d_urn="urn:adsk.eagle:package:25643991/1"/>
-<part name="JP1" library="DoggBone_RC5" library_urn="urn:adsk.eagle:library:25643843" deviceset="JUMPER-SMT_2_NO" device="_SILK" package3d_urn="urn:adsk.eagle:package:25643984/1"/>
-<part name="JP2" library="DoggBone_RC5" library_urn="urn:adsk.eagle:library:25643843" deviceset="JUMPER-SMT_2_NO" device="_SILK" package3d_urn="urn:adsk.eagle:package:25643984/1"/>
-<part name="FRAME2" library="BoardLE+" library_urn="urn:adsk.eagle:library:23298109" deviceset="LETTER_L" device=""/>
-<part name="J1" library="BoardLE+" library_urn="urn:adsk.eagle:library:23298109" deviceset="10118193-0001LF" device=""/>
-<part name="SUPPLY2" library="DoggBone_RC5" library_urn="urn:adsk.eagle:library:25643843" deviceset="V_USB" device=""/>
-<part name="GND2" library="BoardLE+" library_urn="urn:adsk.eagle:library:23298109" deviceset="GND" device=""/>
-<part name="C1" library="BoardLE+" library_urn="urn:adsk.eagle:library:23298109" deviceset="CAP_0.1UF_25V_X7R" device="-0603" package3d_urn="urn:adsk.eagle:package:25646683/2" value="0.1uF"/>
-<part name="C2" library="BoardLE+" library_urn="urn:adsk.eagle:library:23298109" deviceset="CAP_22UF_16V_X5R" device="-0603" package3d_urn="urn:adsk.eagle:package:23298175/3" value="22uF"/>
-<part name="RED" library="SparkFun-LED" deviceset="WS2812" device="_5050"/>
-<part name="GREEN" library="SparkFun-LED" deviceset="WS2812" device="_5050"/>
-<part name="BLUE" library="SparkFun-LED" deviceset="WS2812" device="_5050"/>
-<part name="MIXED" library="SparkFun-LED" deviceset="WS2812" device="_5050"/>
-<part name="GND1" library="BoardLE+" library_urn="urn:adsk.eagle:library:23298109" deviceset="GND" device=""/>
-<part name="SUPPLY3" library="DoggBone_RC5" library_urn="urn:adsk.eagle:library:25643843" deviceset="V_USB" device=""/>
-<part name="C3" library="BoardLE+" library_urn="urn:adsk.eagle:library:23298109" deviceset="CAP_0.1UF_25V_X7R" device="-0603" package3d_urn="urn:adsk.eagle:package:25646683/2" value="0.1uF"/>
-<part name="C4" library="BoardLE+" library_urn="urn:adsk.eagle:library:23298109" deviceset="CAP_0.1UF_25V_X7R" device="-0603" package3d_urn="urn:adsk.eagle:package:25646683/2" value="0.1uF"/>
-<part name="C5" library="BoardLE+" library_urn="urn:adsk.eagle:library:23298109" deviceset="CAP_0.1UF_25V_X7R" device="-0603" package3d_urn="urn:adsk.eagle:package:25646683/2" value="0.1uF"/>
-<part name="C6" library="BoardLE+" library_urn="urn:adsk.eagle:library:23298109" deviceset="CAP_0.1UF_25V_X7R" device="-0603" package3d_urn="urn:adsk.eagle:package:25646683/2" value="0.1uF"/>
-<part name="GND3" library="BoardLE+" library_urn="urn:adsk.eagle:library:23298109" deviceset="GND" device=""/>
-<part name="SUPPLY4" library="DoggBone_RC5" library_urn="urn:adsk.eagle:library:25643843" deviceset="V_USB" device=""/>
-<part name="RED_POT" library="BoardLE+" library_urn="urn:adsk.eagle:library:23298109" deviceset="PTA2043-2015DPB103" device=""/>
-<part name="GREEN_POT" library="BoardLE+" library_urn="urn:adsk.eagle:library:23298109" deviceset="PTA2043-2015DPB103" device=""/>
-<part name="BLUE_POT" library="BoardLE+" library_urn="urn:adsk.eagle:library:23298109" deviceset="PTA2043-2015DPB103" device=""/>
-<part name="GND4" library="BoardLE+" library_urn="urn:adsk.eagle:library:23298109" deviceset="GND" device=""/>
-<part name="SUPPLY5" library="DoggBone_RC5" library_urn="urn:adsk.eagle:library:25643843" deviceset="V_USB" device=""/>
-<part name="GND5" library="BoardLE+" library_urn="urn:adsk.eagle:library:23298109" deviceset="GND" device=""/>
-<part name="J2" library="BoardLE+" library_urn="urn:adsk.eagle:library:23298109" deviceset="CONN_02" device="" package3d_urn="urn:adsk.eagle:package:25908307/6"/>
-<part name="GND6" library="BoardLE+" library_urn="urn:adsk.eagle:library:23298109" deviceset="GND" device=""/>
-<part name="VCC" library="DoggBone_RC5" library_urn="urn:adsk.eagle:library:25643843" deviceset="TEST-POINT" device="40MIL" package3d_urn="urn:adsk.eagle:package:25643991/1"/>
-<part name="GND" library="DoggBone_RC5" library_urn="urn:adsk.eagle:library:25643843" deviceset="TEST-POINT" device="40MIL" package3d_urn="urn:adsk.eagle:package:25643991/1"/>
+<part name="U2" library="Color-Experimentation" deviceset="ATTINY85-20MUR" device=""/>
+<part name="GND14" library="Color-Experimentation" deviceset="GND" device=""/>
+<part name="SUPPLY1" library="Color-Experimentation" deviceset="V_USB" device=""/>
+<part name="SCK" library="Color-Experimentation" deviceset="TEST-POINT" device="40MIL">
+<variant name="DEFAULT" populate="no"/>
+</part>
+<part name="MOSI" library="Color-Experimentation" deviceset="TEST-POINT" device="40MIL">
+<variant name="DEFAULT" populate="no"/>
+</part>
+<part name="MISO" library="Color-Experimentation" deviceset="TEST-POINT" device="40MIL">
+<variant name="DEFAULT" populate="no"/>
+</part>
+<part name="RST" library="Color-Experimentation" deviceset="TEST-POINT" device="40MIL">
+<variant name="DEFAULT" populate="no"/>
+</part>
+<part name="JP1" library="Color-Experimentation" deviceset="JUMPER-SMT_2_NO" device="_SILK">
+<variant name="DEFAULT" populate="no"/>
+</part>
+<part name="JP2" library="Color-Experimentation" deviceset="JUMPER-SMT_2_NO" device="_SILK">
+<variant name="DEFAULT" populate="no"/>
+</part>
+<part name="FRAME2" library="Color-Experimentation" deviceset="LETTER_L" device=""/>
+<part name="J1" library="Color-Experimentation" deviceset="10118193-0001LF" device=""/>
+<part name="SUPPLY2" library="Color-Experimentation" deviceset="V_USB" device=""/>
+<part name="GND2" library="Color-Experimentation" deviceset="GND" device=""/>
+<part name="C1" library="Color-Experimentation" deviceset="CAP_0.1UF_25V_X7R" device="-0603" value="0.1uF"/>
+<part name="C2" library="Color-Experimentation" deviceset="CAP_22UF_16V_X5R" device="-0603" value="22uF"/>
+<part name="RED" library="Color-Experimentation" deviceset="WS2812" device="_5050" value="WS2812"/>
+<part name="GREEN" library="Color-Experimentation" deviceset="WS2812" device="_5050" value="WS2812"/>
+<part name="BLUE" library="Color-Experimentation" deviceset="WS2812" device="_5050" value="WS2812"/>
+<part name="MIXED" library="Color-Experimentation" deviceset="WS2812" device="_5050" value="WS2812"/>
+<part name="GND1" library="Color-Experimentation" deviceset="GND" device=""/>
+<part name="SUPPLY3" library="Color-Experimentation" deviceset="V_USB" device=""/>
+<part name="C3" library="Color-Experimentation" deviceset="CAP_0.1UF_25V_X7R" device="-0603" value="0.1uF"/>
+<part name="C4" library="Color-Experimentation" deviceset="CAP_0.1UF_25V_X7R" device="-0603" value="0.1uF"/>
+<part name="C5" library="Color-Experimentation" deviceset="CAP_0.1UF_25V_X7R" device="-0603" value="0.1uF"/>
+<part name="C6" library="Color-Experimentation" deviceset="CAP_0.1UF_25V_X7R" device="-0603" value="0.1uF"/>
+<part name="GND3" library="Color-Experimentation" deviceset="GND" device=""/>
+<part name="SUPPLY4" library="Color-Experimentation" deviceset="V_USB" device=""/>
+<part name="RED_POT" library="Color-Experimentation" deviceset="PTA2043-2015DPB103" device="" value="10k"/>
+<part name="GREEN_POT" library="Color-Experimentation" deviceset="PTA2043-2015DPB103" device="" value="10k"/>
+<part name="BLUE_POT" library="Color-Experimentation" deviceset="PTA2043-2015DPB103" device="" value="10k"/>
+<part name="GND4" library="Color-Experimentation" deviceset="GND" device=""/>
+<part name="SUPPLY5" library="Color-Experimentation" deviceset="V_USB" device=""/>
+<part name="GND5" library="Color-Experimentation" deviceset="GND" device=""/>
+<part name="J2" library="Color-Experimentation" deviceset="CONN_02" device=""/>
+<part name="GND6" library="Color-Experimentation" deviceset="GND" device=""/>
+<part name="VCC" library="Color-Experimentation" deviceset="TEST-POINT" device="40MIL">
+<variant name="DEFAULT" populate="no"/>
+</part>
+<part name="GND" library="Color-Experimentation" deviceset="TEST-POINT" device="40MIL">
+<variant name="DEFAULT" populate="no"/>
+</part>
 </parts>
 <sheets>
@@
 </schematic>
 </drawing>
-<compatibility>
-<note version="8.2" severity="warning">
-Since Version 8.2, EAGLE supports online libraries. The ids
-of those online libraries will not be understood (or retained)
-with this version.
-</note>
-<note version="8.3" severity="warning">
-Since Version 8.3, EAGLE supports URNs for individual library
-assets (packages, symbols, and devices). The URNs of those assets
-will not be understood (or retained) with this version.
-</note>
-<note version="8.3" severity="warning">
-Since Version 8.3, EAGLE supports the association of 3D packages
-with devices in libraries, schematics, and board files. Those 3D
-packages will not be understood (or retained) with this version.
-</note>
-</compatibility>
 </eagle>

Commit message: Add pullup, solder jumper on "mixed LED enable"
Parts:
- added JP3: JUMPER-SMT_2_NO_SILK, Color-Experimentation:JUMPER-SMT_2_NO_SILK
- added R1: 10k, Color-Experimentation:RES_10K_1%R0603
Connections:
- new net N$3: J2.1, JP3.1, R1.2
- net N$6: now also JP3.2; no longer J2.1
- net V_USB: now also R1.1
Other:
- note added: "After programming, close JP1, JP2, JP3"
- note removed: "After programming, close JP1, JP2"
- moved on the sheet: J2
Changed lines of the file:
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@@
 <variant name="DEFAULT" populate="no"/>
 </part>
+<part name="R1" library="Color-Experimentation" deviceset="RES_10K_1%" device="R0603" package3d_urn="urn:adsk.eagle:package:23298173/3" value="10k"/>
+<part name="SUPPLY6" library="Color-Experimentation" deviceset="V_USB" device=""/>
+<part name="JP3" library="Color-Experimentation" deviceset="JUMPER-SMT_2_NO" device="_SILK"/>
 </parts>
 <sheets>
@@
 <plain>
 <text x="320.04" y="142.24" size="1.778" layer="97">Decoupling Caps</text>
-<text x="449.58" y="106.68" size="1.778" layer="97">After programming, close JP1, JP2</text>
+<text x="449.58" y="106.68" size="1.778" layer="97">After programming, close JP1, JP2, JP3</text>
 <text x="474.98" y="170.18" size="1.778" layer="97">LED Decoupling Caps</text>
 <text x="398.78" y="165.1" size="1.778" layer="97">USB Connector for Power</text>
@@
 <text x="327.66" y="228.6" size="1.778" layer="97">Slider Potentiometers</text>
 <text x="375.92" y="121.92" size="1.778" layer="97">Microcontroller</text>
-<text x="317.5" y="88.9" size="1.778" layer="97">Close J2 to enable MIXED LED</text>
+<text x="317.5" y="68.58" size="1.778" layer="97">Close J2 to enable MIXED LED</text>
 </plain>
 <instances>
@@
 <attribute name="VALUE" x="332.74" y="119.38" size="1.778" layer="96"/>
 </instance>
-<instance part="J2" gate="G$1" x="330.2" y="101.6" smashed="yes">
-<attribute name="VALUE" x="327.66" y="96.774" size="1.778" layer="96" font="vector"/>
-<attribute name="NAME" x="327.66" y="107.188" size="1.778" layer="95" font="vector"/>
-</instance>
-<instance part="GND6" gate="1" x="340.36" y="96.52" smashed="yes">
-<attribute name="VALUE" x="337.82" y="93.98" size="1.778" layer="96"/>
+<instance part="J2" gate="G$1" x="330.2" y="81.28" smashed="yes">
+<attribute name="VALUE" x="327.66" y="76.454" size="1.778" layer="96" font="vector"/>
+<attribute name="NAME" x="327.66" y="86.868" size="1.778" layer="95" font="vector"/>
+</instance>
+<instance part="GND6" gate="1" x="340.36" y="76.2" smashed="yes">
+<attribute name="VALUE" x="337.82" y="73.66" size="1.778" layer="96"/>
 </instance>
 <instance part="VCC" gate="G$1" x="441.96" y="165.1" smashed="yes">
@@
 <instance part="GND" gate="G$1" x="441.96" y="144.78" smashed="yes">
 <attribute name="NAME" x="447.04" y="144.78" size="1.778" layer="95" font="vector"/>
+</instance>
+<instance part="R1" gate="G$1" x="332.74" y="93.98" smashed="yes">
+<attribute name="NAME" x="328.93" y="95.4786" size="1.778" layer="95"/>
+<attribute name="VALUE" x="328.93" y="90.678" size="1.778" layer="96"/>
+</instance>
+<instance part="SUPPLY6" gate="G$1" x="325.12" y="99.06" smashed="yes">
+<attribute name="VALUE" x="325.12" y="101.854" size="1.778" layer="96" align="bottom-center"/>
+</instance>
+<instance part="JP3" gate="G$1" x="340.36" y="101.6" smashed="yes" rot="R90">
+<attribute name="NAME" x="337.82" y="99.06" size="1.778" layer="95" font="vector" rot="R90"/>
 </instance>
 </instances>
@@
 <segment>
 <pinref part="J2" gate="G$1" pin="2"/>
-<wire x1="337.82" y1="101.6" x2="340.36" y2="101.6" width="0.1524" layer="91"/>
+<wire x1="337.82" y1="81.28" x2="340.36" y2="81.28" width="0.1524" layer="91"/>
 <pinref part="GND6" gate="1" pin="GND"/>
-<wire x1="340.36" y1="101.6" x2="340.36" y2="99.06" width="0.1524" layer="91"/>
+<wire x1="340.36" y1="81.28" x2="340.36" y2="78.74" width="0.1524" layer="91"/>
 </segment>
 </net>
@@
 <pinref part="SUPPLY5" gate="G$1" pin="V_USB"/>
 </segment>
+<segment>
+<pinref part="R1" gate="G$1" pin="1"/>
+<wire x1="327.66" y1="93.98" x2="325.12" y2="93.98" width="0.1524" layer="91"/>
+<wire x1="325.12" y1="93.98" x2="325.12" y2="99.06" width="0.1524" layer="91"/>
+<pinref part="SUPPLY6" gate="G$1" pin="V_USB"/>
+</segment>
 </net>
 <net name="LED_DATA_OUT" class="0">
@@
 <segment>
 <pinref part="U2" gate="A" pin="PB1(MISO/PCINT1)"/>
-<wire x1="340.36" y1="111.76" x2="355.6" y2="111.76" width="0.1524" layer="91"/>
 <pinref part="MISO" gate="G$1" pin="1"/>
+<wire x1="355.6" y1="111.76" x2="340.36" y2="111.76" width="0.1524" layer="91"/>
+<pinref part="JP3" gate="G$1" pin="2"/>
 <wire x1="340.36" y1="111.76" x2="314.96" y2="111.76" width="0.1524" layer="91"/>
+<wire x1="340.36" y1="106.68" x2="340.36" y2="111.76" width="0.1524" layer="91"/>
 <junction x="340.36" y="111.76"/>
+</segment>
+</net>
+<net name="N$3" class="0">
+<segment>
+<pinref part="R1" gate="G$1" pin="2"/>
+<wire x1="337.82" y1="93.98" x2="340.36" y2="93.98" width="0.1524" layer="91"/>
+<wire x1="340.36" y1="83.82" x2="340.36" y2="93.98" width="0.1524" layer="91"/>
 <pinref part="J2" gate="G$1" pin="1"/>
-<wire x1="337.82" y1="104.14" x2="340.36" y2="104.14" width="0.1524" layer="91"/>
-<wire x1="340.36" y1="104.14" x2="340.36" y2="111.76" width="0.1524" layer="91"/>
+<wire x1="337.82" y1="83.82" x2="340.36" y2="83.82" width="0.1524" layer="91"/>
+<pinref part="JP3" gate="G$1" pin="1"/>
+<wire x1="340.36" y1="93.98" x2="340.36" y2="96.52" width="0.1524" layer="91"/>
+<junction x="340.36" y="93.98"/>
 </segment>
 </net>
@@
 </schematic>
 </drawing>
+<compatibility>
+<note version="8.3" severity="warning">
+Since Version 8.3, EAGLE supports URNs for individual library
+assets (packages, symbols, and devices). The URNs of those assets
+will not be understood (or retained) with this version.
+</note>
+<note version="8.3" severity="warning">
+Since Version 8.3, EAGLE supports the association of 3D packages
+with devices in libraries, schematics, and board files. Those 3D
+packages will not be understood (or retained) with this version.
+</note>
+</compatibility>
 </eagle>

Commit message: add attribution to sch
Other:
- note added: "Jonathan Moyes"
Changed lines of the file:
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@@
 <text x="375.92" y="121.92" size="1.778" layer="97">Microcontroller</text>
 <text x="317.5" y="68.58" size="1.778" layer="97">Close J2 to enable MIXED LED</text>
+<text x="431.8" y="78.74" size="3.81" layer="94">Jonathan Moyes</text>
 </plain>
 <instances>
